File: board/RISKYMouse.kicad_sch (KiCad schematic)
At the start: 18 parts, among them J1 USB_1, J3 Conn_01x02, J4 DE9_Plug, U1 CH32V203C8T6, U2 LM1117MP-3.3

Commit message: New PCB design
Parts:
- removed C7: 0.1μF, Capacitor_SMD:C_0603_1608Metric_Pad1.08x0.95mm_HandSolder, symbol Device:C_Small
- removed J1: USB_1, Connector_USB:USB_A_CONNFLY_DS1095-WNR0, symbol Connector:USB_A
- removed J3: Conn_01x02, Connector_PinHeader_2.54mm:PinHeader_1x02_P2.54mm_Vertical, symbol Connector_Generic:Conn_01x02
- removed J4: DE9_Plug, Connector_Dsub:DSUB-9_Female_EdgeMount_P2.77mm, symbol Connector:DE9_Plug
- added C9: 0.1μF, Capacitor_SMD:C_0603_1608Metric_Pad1.08x0.95mm_HandSolder, symbol Device:C_Small
- added D3: LED, LED_SMD:LED_0805_2012Metric_Pad1.15x1.40mm_HandSolder, symbol Device:LED
- added J1: DE9_Plug, Connector_Dsub:DSUB-9_Female_EdgeMount_P2.77mm, symbol Connector:DE9_Plug
- added J2: Conn_01x02, Connector_PinHeader_2.54mm:PinHeader_1x02_P2.54mm_Vertical, symbol Connector_Generic:Conn_01x02
- added J3: USB_1, Connector_USB:USB_A_CONNFLY_DS1095-WNR0, symbol Connector:USB_A
- added R4: 2.2k, Resistor_SMD:R_0603_1608Metric_Pad0.98x0.95mm_HandSolder, symbol Device:R
Connections:
- net +3.3V: now also R4.2
- net +5V: now also J1.7
- net GND: now also C9.2, J1.8, J3.4 (GND), J3.5 (Shield)
- net NRST: now also C9.1
- net PIN1: now also J1.1
- net PIN2: now also J1.2
- net PIN3: now also J1.3
- net PIN4: now also J1.4
- net PIN5: now also J1.5
- net PIN6: now also J1.6
- net PIN9: now also J1.9
- net SWCLK: now also J2.1 (Pin_1)
- net SWDIO: now also J2.2 (Pin_2)
- net USB_DM: now also J3.2 (D-)
- net USB_DP: now also J3.3 (D+)
- net at F1.1: now also J3.1 (VBUS)
- net LED2: now reaches U1.4 (PC15_OSC32OUT)
- net LED2: now also D3.1 (K)
- new net: D3.2 (A), R4.1
- no-connect marks 24 -> 23
